Commit message: working flat

File: exts/trace_humanoid/trace_humanoid/assets/Robots/humanoid/humanoid_urdf/urdf/humanoid_urdf.urdf (robot description, URDF)
Before this commit: robot humanoid_urdf, 11 links, 10 joints
Links:
- link left_knee_link: geometry collision mesh filename=../meshes/knee_collision.STL; visual mesh filename=../meshes/left_knee_link.STL
- link right_knee_link: geometry collision mesh filename=../meshes/knee_collision.STL; visual mesh filename=../meshes/right_knee_link.STL
